Commit message: ajusted xacro and added session

File: blue/models/mrs_robots_description/urdf/blue.xacro (robot description, xacro)
@@ -407,14 +407,14 @@
       <origin xyz="0 0 0" rpy="0 0 0" />
     </xacro:visual_macro>
-    <!-- <xacro:visual_macro_common_geometry_type -->
-    <!--   robot_namespace="${namespace}" -->
-    <!--   name="battery" -->
-    <!--   parent="base_link" -->
-    <!--   color="Grey"> -->
-    <!--   <origin xyz="0.0 0 -${0.45*body_height}" rpy="0 0 0" /> -->
-    <!--   <geometry> -->
-    <!--     <box size="0.16 0.065 0.044" /> -->
-    <!--   </geometry> -->
-    <!-- </xacro:visual_macro_common_geometry_type> -->
+    <xacro:visual_macro_common_geometry_type
+      robot_namespace="${namespace}"
+      name="battery"
+      parent="base_link"
+      color="black">
+      <origin xyz="0.0 0 -${0.45*body_height}" rpy="0 0 0" />
+      <geometry>
+        <box size="0.132 0.042 0.044" />
+      </geometry>
+    </xacro:visual_macro_common_geometry_type>
   </xacro:if>
   <!--}-->

Commit message: added rplidar

File: blue/models/mrs_robots_description/urdf/blue.xacro (robot description, xacro)
@@ -411,5 +411,5 @@
       name="battery"
       parent="base_link"
-      color="black">
+      color="Black">
       <origin xyz="0.0 0 -${0.45*body_height}" rpy="0 0 0" />
       <geometry>
@@ -570,4 +570,26 @@
   <!--}-->
   <!--} Bluefox placements-->
+  <!-- ========================== LIDAR sensors ========================= -->
+  <!-- Rplidar {-->
+  <xacro:rplidar_macro
+    namespace="${namespace}"
+    x="0.0"
+    y="0.0"
+    z="0.127"
+    roll="0"
+    pitch="0"
+    yaw="0"
+    >
+  </xacro:rplidar_macro>
+  <xacro:visual_macro
+    robot_namespace="${namespace}"
+    name="rplidar_mount"
+    mesh_file="${rplidar_mount_mesh}"
+    mesh_scale="${mesh_scale}"
+    parent="base_link"
+    color="Blue">
+    <origin xyz="0 0 0" rpy="0 0 0" />
+  </xacro:visual_macro>
+  <!--}-->
   <!-- ================================================================== -->
   <!-- ||                      external parts                          || -->

Commit message: fixed gripper friction

File: blue/models/mrs_robots_description/urdf/blue.xacro (robot description, xacro)
@@ -75,5 +75,5 @@
   <xacro:property name="rplidar_mount_mesh" value="package://mrs_robots_description/meshes/holybro_x500_rplidar_mount.dae" />
   <!-- external parts -->
-  <xacro:property name="grip_mesh_file" value="package://mrs_robots_description/meshes/holybro_x500_grip.dae" />
+  <xacro:property name="grip_mesh_file" value="package://mrs_robots_description/meshes/holybro_x500_grip1.dae" />
   <!-- scales -->
   <xacro:property name="mesh_scale" value="1 1 1"/>
@@ -606,9 +606,9 @@
     joint="continuous"
     axis="1 0 0"
-    damping="0.7"
-    friction="0.7"
-    upper="0.04"
-    lower="0.0"
-    effort="20"
+    damping="0.1"
+    friction="0.9"
+    upper="0.1"
+    lower="0.04"
+    effort="50000000"
     velocity="0.2"
     mass="0.033912"
@@ -631,9 +631,9 @@
     joint="continuous"
     axis="1 0 0"
-    damping="0.7"
-    friction="0.7"
-    upper="0.04"
-    lower="0.0"
-    effort="20"
+    damping="0.1"
+    friction="0.9"
+    upper="0.1"
+    lower="0.04"
+    effort="50000000"
     velocity="0.2"
     mass="0.033912"

File: blue/models/mrs_robots_description/urdf/component_snippets.xacro (robot description, xacro)
@@ -185,5 +185,5 @@
               <ode>
                 <mu>100</mu>
-                <mu2>100</mu2>
+                <mu2>0.9</mu2>
               </ode>
             </friction>
@@ -196,6 +196,6 @@
       </link>
       <gazebo reference="${name}_link">
-        <mu1>100</mu1>
-        <mu2>100</mu2>
+        <mu1>0.9</mu1>
+        <mu2>0.9</mu2>
         <material>Gazebo/${color}</material>
       </gazebo>

Commit message: fixed gripper

File: blue/models/mrs_robots_description/urdf/blue.xacro (robot description, xacro)
@@ -620,5 +620,5 @@
     izz="0.000082322785"
     color="Blue">
-    <origin xyz="0.0 0.0 0.0" rpy="0 0 0" />
+    <origin xyz="0.0 0.0 0.01" rpy="0 0 0" />
   </xacro:visual_macro_with_collision_joint>
   <!-- grip right visual {-->
@@ -645,5 +645,5 @@
     izz="0.000082322785"
     color="Blue">
-    <origin xyz="0.0 0.0 0.0" rpy="0 0 ${rad180}" />
+    <origin xyz="0.0 0.0 0.01" rpy="0 0 ${rad180}" />
   </xacro:visual_macro_with_collision_joint>
   <xacro:transmissions_joints

Commit message: added realsense down

File: blue/models/mrs_robots_description/urdf/blue.xacro (robot description, xacro)
@@ -534,8 +534,8 @@
   <!--}-->
   <!-- Realsense front {-->
-  <xacro:realsense_macro
+  <xacro:realsenseD435_macro
     namespace="${namespace}"
     camera_name="rgbd"
-    camera_suffix=""
+    camera_suffix="front"
     parent_link="base_link"
     parent_frame_name="${namespace}/fcu"
@@ -547,28 +547,22 @@
     pitch="0"
     yaw="0">
-  </xacro:realsense_macro>
-  <!--}-->
-  <!-- Bluefox placements{-->
-  <!-- classic {-->
-  <xacro:bluefox_camera_macro
-    namespace="${namespace}"
+  </xacro:realsenseD435_macro>
+  <!--}-->
+    <!-- Realsense down {-->
+  <xacro:realsenseD455_macro
+    namespace="${namespace}"
+    camera_name="rgbd"
+    camera_suffix="down"
     parent_link="base_link"
-    camera_suffix="bluefox_optflow"
-    frame_rate="100.0"
-    hfov="2.1"
-    noise="0.007"
     parent_frame_name="${namespace}/fcu"
-    camera_frame_name="${namespace}/bluefox_optflow_optical"
-    sensor_base_frame_name="${namespace}/bluefox_optflow"
-    x="0.08"
+    enable_realistic_realsense="true"
+    x="0.085"
     y="0.00"
-    z="-0.05"
+    z="-0.03"
     roll="0"
     pitch="${rad90}"
-    yaw="0"
-    >
-  </xacro:bluefox_camera_macro>
-  <!--}-->
-  <!--} Bluefox placements-->
+    yaw="0">
+  </xacro:realsenseD455_macro>
+  <!--}-->
   <!-- ========================== LIDAR sensors ========================= -->
   <!-- Rplidar {-->

File: blue/models/mrs_robots_description/urdf/component_snippets.xacro (robot description, xacro)
@@ -1712,5 +1712,5 @@
   <!-- ========================= camera sensors ========================= -->
   <!-- Macro to add an Intel Realsense D435 {-->
-  <xacro:macro name="realsense_macro"
+  <xacro:macro name="realsenseD435_macro"
     params="namespace camera_name parent_link parent_frame_name camera_suffix x y z roll pitch yaw enable_realistic_realsense">
     <!-- visual links and joints {-->
@@ -1906,4 +1906,199 @@
   </xacro:macro>
   <!--}-->
+  <!-- Macro to add an Intel Realsense D455 {-->
+  <xacro:macro name="realsenseD455_macro"
+    params="namespace camera_name parent_link parent_frame_name camera_suffix x y z roll pitch yaw enable_realistic_realsense">
+    <!-- visual links and joints {-->
+    <link name="${camera_name}/camera${camera_suffix}">
+      <visual>
+        <origin xyz="0.0 0.0 0" rpy="-${rad90} 0 -${rad90}" />
+        <geometry>
+          <mesh filename="package://mrs_robots_description/meshes/sensors/realsense_body.stl"
+            scale="0.001 0.001 0.001" />
+        </geometry>
+      </visual>
+    </link>
+    <link name="${camera_name}/camera${camera_suffix}_glass_link">
+      <visual>
+        <origin xyz="0.0 0.0 0" rpy="-${rad90} 0 -${rad90}" />
+        <geometry>
+          <mesh filename="package://mrs_robots_description/meshes/sensors/realsense_glass.stl"
+            scale="0.001 0.001 0.001" />
+        </geometry>
+      </visual>
+    </link>
+    <joint name="${camera_name}/camera${camera_suffix}_joint" type="fixed">
+      <origin xyz="${x} ${y} ${z}" rpy="${roll} ${pitch} ${yaw}"/>
+      <parent link="${parent_link}" />
+      <child link="${camera_name}/camera${camera_suffix}" />
+    </joint>
+    <joint name="${camera_name}/camera${camera_suffix}_glass_joint" type="fixed">
+      <origin xyz="0 0 0 " rpy="0 0 0"/>
+      <parent link="${camera_name}/camera${camera_suffix}" />
+      <child link="${camera_name}/camera${camera_suffix}_glass_link" />
+    </joint>
+    <!--}-->
+    <gazebo>
+      <plugin name="${camera_name}${camera_suffix}_plugin" filename="libMRSGazeboRealsensePlugin.so">
+        <camera_name>${camera_name}</camera_name>
+        <camera_suffix>${camera_suffix}</camera_suffix>
+        <useRealistic>${enable_realistic_realsense}</useRealistic>
+        <noisePerMeter>0.2</noisePerMeter>
+        <minNoiseDistance>4.0</minNoiseDistance>
+        <perlinEmptyThreshold>0.8</perlinEmptyThreshold>
+        <perlinEmptySpeed>0.2</perlinEmptySpeed>
+        <imageScaling>4</imageScaling>
+        <blurSize>15</blurSize>
+        <erosionSize>5</erosionSize>
+        <parentFrameName>${parent_frame_name}</parentFrameName>
+        <x>${x}</x>
+        <y>${y}</y>
+        <z>${z}</z>
+        <roll>${roll}</roll>
+        <pitch>${pitch}</pitch>
+        <yaw>${yaw}</yaw>
+      </plugin>
+    </gazebo>
+    <!-- sensors {-->
+    <gazebo reference="${camera_name}/camera${camera_suffix}">
+      <!-- rgb camera {-->
+      <sensor name="${namespace}/${camera_name}${camera_suffix}_color" type="camera">
+        <!-- <pose frame="">0 -0.046 0.004 0 0 0</pose> -->
+        <pose frame="">0 0 -0.0115 0 0 0</pose>
+        <camera name="${camera_name}${camera_suffix}/camera">
+          <!-- <horizontal_fov>1.211259</horizontal_fov> -->
+          <horizontal_fov>1.5708</horizontal_fov>
+          <image>
+            <width>1280</width>
+            <height>800</height>
+            <format>RGB_INT8</format>
+          </image>
+          <clip>
+            <near>0.1</near>
+            <far>100</far>
+          </clip>
+          <noise>
+            <type>gaussian</type>
+            <mean>0.0</mean>
+            <stddev>0.007</stddev>
+          </noise>
+        </camera>
+        <always_on>1</always_on>
+        <update_rate>60</update_rate>
+        <visualize>0</visualize>
+      </sensor>
+      <!--}-->
+      <!-- infra stereo {-->
+      <sensor name="${namespace}/${camera_name}${camera_suffix}_infra_stereo" type="multicamera">
+        <always_on>1</always_on>
+        <update_rate>30</update_rate>
+        <visualize>0</visualize>
+        <camera name="${namespace}/${camera_name}${camera_suffix}/infra1">
+          <!-- <horizontal_fov>1.7523106</horizontal_fov> -->
+          <horizontal_fov>1.211259</horizontal_fov>
+          <image>
+            <width>640</width>
+            <height>360</height>
+            <format>L_INT8</format>
+          </image>
+          <clip>
+            <near>0.1</near>
+            <far>50</far>
+          </clip>
+          <noise>
+            <type>gaussian</type>
+            <mean>0.0</mean>
+            <stddev>0.005</stddev>
+          </noise>
+        </camera>
+        <camera name="${namespace}/${camera_name}${camera_suffix}/infra2">
+          <pose>0 0.05 0 0 0 0</pose>
+          <!-- <horizontal_fov>1.7523106</horizontal_fov> -->
+          <horizontal_fov>1.5708</horizontal_fov>
+          <image>
+            <width>640</width>
+            <height>360</height>
+            <format>L_INT8</format>
+          </image>
+          <clip>
+            <near>0.1</near>
+            <far>50</far>
+          </clip>
+          <noise>
+            <type>gaussian</type>
+            <mean>0.0</mean>
+            <stddev>0.005</stddev>
+          </noise>
+        </camera>
+      </sensor>
+      <!--}-->
+      <!-- (unused) infra2 {-->
+        <!-- <sensor name="infra2" type="camera"> -->
+        <!-- <parent link="${camera_name}${camera_suffix}_camera_${camera_suffix}"/> -->
+        <!-- <pose>0 -1.0325 0 0 0 0</pose> -->
+        <!--   <pose frame="${camera_name}${camera_suffix}/camera_infra2">0 -1.0325 0 0 0 0</pose> -->
+        <!--   <camera name="${camera_name}${camera_suffix}/camera_${camera_suffix}_infra2"> -->
+          <!-- <horizontal_fov>1.7523106</horizontal_fov> -->
+          <!--     <horizontal_fov>1.211259</horizontal_fov> -->
+          <!--     <image> -->
+            <!--       <width>1280</width> -->
+            <!--       <height>720</height> -->
+            <!--       <format>L_INT8</format> -->
+            <!--     </image> -->
+          <!--     <clip> -->
+            <!--       <near>0.1</near> -->
+            <!--       <far>10</far> -->
+            <!--     </clip> -->
+          <!--     <noise> -->
+            <!--       <type>gaussian</type> -->
+            <!--       <mean>0.0</mean> -->
+            <!--       <stddev>0.05</stddev> -->
+            <!--     </noise> -->
+          <!--   </camera> -->
+        <!--   <always_on>1</always_on> -->
+        <!--   <update_rate>60</update_rate> -->
+        <!--   <visualize>0</visualize> -->
+          <!-- </sensor> -->
+          <!--}-->
+      <!-- aligned depth to color {-->
+        <sensor name="${namespace}/${camera_name}${camera_suffix}_aligned_depth_to_color" type="depth">
+        <pose>0 -0.0115 0.0 0 0 0</pose>
+        <camera name="${camera_name}/camera${camera_suffix}">
+          <horizontal_fov>1.211259</horizontal_fov>
+          <image>
+            <xacro:if value="${enable_realistic_realsense}">
+              <width>320</width>
+              <height>180</height>
+            </xacro:if>
+            <xacro:unless value="${enable_realistic_realsense}">
+              <width>1280</width>
+              <height>720</height>
+            </xacro:unless>
+          </image>
+          <clip>
+            <near>0.3</near>
+            <far>12</far>
+          </clip>
+          <noise>
+            <type>gaussian</type>
+            <mean>0.0</mean>
+            <stddev>5000.0</stddev>
+          </noise>
+        </camera>
+        <always_on>1</always_on>
+        <update_rate>60</update_rate>
+        <visualize>0</visualize>
+      </sensor>
+      <!--}-->
+    </gazebo>
+    <!--}-->
+    <gazebo reference="${camera_name}/camera${camera_suffix}">
+      <material>Gazebo/White</material>
+    </gazebo>
+    <gazebo reference="${camera_name}/camera${camera_suffix}_glass_link">
+      <material>Gazebo/BlackTransparent</material>
+    </gazebo>
+  </xacro:macro>
+  <!--}-->
   <!-- Macro to add a Bluefox camera {-->
   <xacro:macro name="bluefox_camera_macro"
